File: Kicad/TestBoard.sch (KiCad schematic (older format))
At the start: 22 parts, among them P1 TST, P2 TST, P3 TST, P4 CONN_4, P5 CONN_2

Commit message: actualizo después de muuucho tiempo archivos no incluidos
Parts:
- C1, C3, C4, C5: symbol CP -> CP-RESCUE-TestBoard
- C2: symbol C -> C-RESCUE-TestBoard
- R1, R2, R3: symbol R -> R-RESCUE-TestBoard
- RV1, RV2, RV3: symbol POT -> POT-RESCUE-TestBoard
Changed lines of the file:
@@
 EESchema Schematic File Version 2
+LIBS:TestBoard-rescue
 LIBS:power
 LIBS:device
@@
 LIBS:memory
 LIBS:xilinx
-LIBS:special
 LIBS:microcontrollers
 LIBS:dsp
@@
 LIBS:74HC132
 LIBS:TestBoard-cache
-EELAYER 27 0
+EELAYER 25 0
 EELAYER END
 $Descr A4 11693 8268
@@
 $EndDescr
 $Comp
-L POT RV1
+L POT-RESCUE-TestBoard RV1
 U 1 1 57910F36
 P 2100 1350
@@
 $EndComp
 $Comp
-L GNDA #PWR01
+L GNDA-RESCUE-TestBoard #PWR01
 U 1 1 57910FFB
 P 2100 2250
@@
 	2100 800  2100 1100
 $Comp
-L R R1
+L R-RESCUE-TestBoard R1
 U 1 1 5791107C
 P 2650 1350
@@
 	2250 1350 2400 1350
 $Comp
-L CP C3
+L CP-RESCUE-TestBoard C3
 U 1 1 57911112
 P 3000 1700
@@
 $EndComp
 $Comp
-L GNDA #PWR05
+L GNDA-RESCUE-TestBoard #PWR05
 U 1 1 57963C51
 P 1250 3150
@@
 $EndComp
 $Comp
-L CP C1
+L CP-RESCUE-TestBoard C1
 U 1 1 57963C5A
 P 1250 2750
@@
 	1250 2950 1250 3150
 $Comp
-L C C2
+L C-RESCUE-TestBoard C2
 U 1 1 57963C81
 P 1600 2750
@@
 Connection ~ 1250 3000
 $Comp
-L POT RV2
+L POT-RESCUE-TestBoard RV2
 U 1 1 57963E06
 P 2100 3250
@@
 $EndComp
 $Comp
-L GNDA #PWR06
+L GNDA-RESCUE-TestBoard #PWR06
 U 1 1 57963E0F
 P 2100 4150
@@
 	2100 2700 2100 3000
 $Comp
-L R R2
+L R-RESCUE-TestBoard R2
 U 1 1 57963E24
 P 2650 3250
@@
 	2250 3250 2400 3250
 $Comp
-L CP C4
+L CP-RESCUE-TestBoard C4
 U 1 1 57963E2E
 P 3000 3600
@@
 ADC1
 $Comp
-L POT RV3
+L POT-RESCUE-TestBoard RV3
 U 1 1 57963E5A
 P 2100 5250
@@
 $EndComp
 $Comp
-L GNDA #PWR09
+L GNDA-RESCUE-TestBoard #PWR09
 U 1 1 57963E63
 P 2100 6150
@@
 	2100 4700 2100 5000
 $Comp
-L R R3
+L R-RESCUE-TestBoard R3
 U 1 1 57963E78
 P 2650 5250
@@
 	2250 5250 2400 5250
 $Comp
-L CP C5
+L CP-RESCUE-TestBoard C5
 U 1 1 57963E82
 P 3000 5600
